Commit message: Fixed the transform from the UR in order for the original pick and place demo to work

File: ur_custom_pkg/urdf/test_ur5e.xacro (robot description, xacro)
@@ -343,5 +343,5 @@
         <parent link="world"/>
         <child link="base_link"/>
-        <origin rpy="0 0 0" xyz="0 0 0.6"/>
+        <origin rpy="0 0 0" xyz="0 0 0"/>
     </joint>
     <!-- ROS-Industrial 'flange' frame: attachment point for EEF models -->
